File: Eagle/StackBreakout/StackBreakoutConnection_4layers_V1.0_with_connector/StackBreakoutConnection_4layers_V1.0_with_connector.sch (EAGLE design)
At the start: 6 parts, among them J1 SSQ-126-23-G-D, J2 SSQ-126-23-G-D, J3 SSQ-126-23-G-D, J4 SSQ-126-23-G-D, X1 53261-06, X2 53261-08

Commit message: Corrección de Aux_x
Connections:
- removed net AUX1: J1B.37, J3B.37
- removed net AUX2: J1B.38, J3B.38
- removed net AUX3: J1B.39, J3B.39
- removed net AUX4: J1B.40, J3B.40
- net AUX_1: now also J1B.37, J3B.37
- net AUX_2: now also J1B.38, J3B.38
- net AUX_3: now also J1B.39, J3B.39
- net AUX_4: now also J1B.40, J3B.40
Changed lines of the file:
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@@
 </segment>
 </net>
-<net name="AUX1" class="0">
+<net name="AUX_1" class="0">
 <segment>
 <pinref part="J1" gate="B" pin="37"/>
@@
 </segment>
 </net>
-<net name="AUX3" class="0">
+<net name="AUX_3" class="0">
 <segment>
 <pinref part="J1" gate="B" pin="39"/>
@@
 </segment>
 </net>
-<net name="AUX2" class="0">
+<net name="AUX_2" class="0">
 <segment>
 <pinref part="J1" gate="B" pin="38"/>
@@
 </segment>
 </net>
-<net name="AUX4" class="0">
+<net name="AUX_4" class="0">
 <segment>
 <pinref part="J1" gate="B" pin="40"/>
